File: pcb/shieldboard/shieldboard.kicad_pcb (KiCad board)
At the start: 2 copper layers, 0 parts

Commit message: pcb: update
Signed-off-by: Ilya Kuzmin <kuzmin.ilya@gmail.com>
Parts:
- added C1: 470,0x16, Capacitor_THT:CP_Radial_D22.0mm_P10.00mm_SnapIn, F.Cu at (67.0, 66.0)
- added C2: 0,1, Capacitor_SMD:C_0805_2012Metric_Pad1.29x1.40mm_HandSolder, F.Cu at (62.0, 47.0)
- added C3: 0,1, Capacitor_SMD:C_0805_2012Metric_Pad1.29x1.40mm_HandSolder, F.Cu at (54.0, 95.5)
- added C4: 0,1, Capacitor_SMD:C_0805_2012Metric_Pad1.29x1.40mm_HandSolder, F.Cu at (54.0, 91.5)
- added C5: 10,0x16, Capacitor_THT:CP_Radial_D13.0mm_P5.00mm, F.Cu at (62.0, 96.0)
- added D1: D, Diode_SMD:D_SMA_Handsoldering, F.Cu at (59.5, 162.0)
- added D2: D, Diode_SMD:D_SMA_Handsoldering, F.Cu at (60.0, 147.0)
- added D3: D, Diode_SMD:D_SMA_Handsoldering, F.Cu at (60.0, 132.0)
- added D4: D, Diode_SMD:D_SMA_Handsoldering, F.Cu at (59.5, 117.0)
- added J1: Conn_01x02, TerminalBlock:TerminalBlock_bornier-2_P5.08mm, F.Cu at (57.0, 46.0)
- added J10: Conn_01x06, Connector_PinHeader_2.54mm:PinHeader_1x06_P2.54mm_Vertical, F.Cu at (82.1, 161.0)
- added J11: Conn_01x18, Connector_PinHeader_2.54mm:PinHeader_1x18_P2.54mm_Vertical, F.Cu at (72.0, 151.3)
- added J12: USB_B, Connector_USB:USB_B_OST_USB-B1HSxx_Horizontal, F.Cu at (102.0, 121.0)
- added J13: Conn_01x01, Connector_Wire:SolderWirePad_1x01_Drill1mm, F.Cu at (101.0, 112.0)
- added J2: Conn_01x02, TerminalBlock:TerminalBlock_bornier-2_P5.08mm, F.Cu at (67.0, 46.0)
- added J3: Conn_01x02, TerminalBlock:TerminalBlock_bornier-2_P5.08mm, F.Cu at (58.0, 156.0)
- added J4: Conn_01x02, TerminalBlock:TerminalBlock_bornier-2_P5.08mm, F.Cu at (58.0, 141.0)
- added J5: Conn_01x02, TerminalBlock:TerminalBlock_bornier-2_P5.08mm, F.Cu at (58.0, 126.0)
- added J6: Conn_01x02, TerminalBlock:TerminalBlock_bornier-2_P5.08mm, F.Cu at (58.0, 111.0)
- added J7: Conn_01x02, TerminalBlock:TerminalBlock_bornier-2_P5.08mm, F.Cu at (62.0, 83.0)
- added J8: Conn_01x06, Connector_PinHeader_2.54mm:PinHeader_1x06_P2.54mm_Vertical, F.Cu at (100.6, 161.0)
- added J9: Conn_01x07, Connector_PinHeader_2.54mm:PinHeader_1x07_P2.54mm_Vertical, F.Cu at (79.5, 96.0)
- added M1: LM2596_DC-DC_module, ki_modules:LM2596_DC-DC_module, F.Cu at (87.0, 66.0)
- added M2: Maple_Mini, ki_modules:Maple_Mini, F.Cu at (87.0, 131.0)
- added Q1: Q_NMOS_GDS, Package_TO_SOT_THT:TO-220-3_Vertical, F.Cu at (50.0, 158.5)
- added Q2: Q_NMOS_GDS, Package_TO_SOT_THT:TO-220-3_Vertical, F.Cu at (50.0, 143.5)
- added Q3: Q_NMOS_GDS, Package_TO_SOT_THT:TO-220-3_Vertical, F.Cu at (50.0, 128.5)
- added Q4: Q_NMOS_GDS, Package_TO_SOT_THT:TO-220-3_Vertical, F.Cu at (50.0, 113.5)
- added R1: 100, Resistor_SMD:R_0805_2012Metric_Pad1.29x1.40mm_HandSolder, F.Cu at (61.0, 166.0)
- added R2: 100, Resistor_SMD:R_0805_2012Metric_Pad1.29x1.40mm_HandSolder, F.Cu at (54.0, 150.0)
- added R3: 100, Resistor_SMD:R_0805_2012Metric_Pad1.29x1.40mm_HandSolder, F.Cu at (54.0, 135.0)
- added R4: 100, Resistor_SMD:R_0805_2012Metric_Pad1.29x1.40mm_HandSolder, F.Cu at (54.0, 120.0)
- added R5: 1,5k, Resistor_SMD:R_0805_2012Metric_Pad1.29x1.40mm_HandSolder, F.Cu at (102.0, 139.0)
- added R6: 22, Resistor_SMD:R_0805_2012Metric_Pad1.15x1.40mm_HandSolder, F.Cu at (102.0, 136.0)
- added R7: 22, Resistor_SMD:R_0805_2012Metric_Pad1.15x1.40mm_HandSolder, F.Cu at (102.0, 133.0)
- added REF**: MountingHole_3.2mm_M3_Pad, MountingHole:MountingHole_3.2mm_M3_Pad, F.Cu at (52.0, 41.0)
- added REF**: MountingHole_3.2mm_M3_Pad, MountingHole:MountingHole_3.2mm_M3_Pad, F.Cu at (107.0, 41.0)
- added REF**: MountingHole_3.2mm_M3_Pad, MountingHole:MountingHole_3.2mm_M3_Pad, F.Cu at (107.0, 141.0)
- added REF**: MountingHole_3.2mm_M3_Pad, MountingHole:MountingHole_3.2mm_M3_Pad, F.Cu at (107.0, 106.0)
- added REF**: MountingHole_3.2mm_M3_Pad, MountingHole:MountingHole_3.2mm_M3_Pad, F.Cu at (52.0, 166.0)
- added REF**: MountingHole_3.2mm_M3_Pad, MountingHole:MountingHole_3.2mm_M3_Pad, F.Cu at (107.0, 166.0)
- added U1: LM7805_TO220, Package_TO_SOT_THT:TO-220-3_Vertical, F.Cu at (50.0, 96.0)
Routing:
- net GND: track 0.00 -> 234.8 mm, vias 0 -> 2
- net +12V: track 0.00 -> 227.8 mm
- net +5V: track 0.00 -> 199.0 mm
- net Net-(M2-PadB8): track 0.00 -> 72.7 mm, vias 0 -> 1
- net Net-(M2-PadB9): track 0.00 -> 60.1 mm, vias 0 -> 1
- net Net-(M2-PadA9): track 0.00 -> 55.2 mm, vias 0 -> 3
- net Net-(M2-PadA8): track 0.00 -> 50.6 mm, vias 0 -> 2
- net Net-(J10-Pad3): track 0.00 -> 49.6 mm, vias 0 -> 1
- net Net-(J10-Pad2): track 0.00 -> 45.2 mm, vias 0 -> 1
- net Net-(J9-Pad1): track 0.00 -> 42.6 mm
- net Net-(J9-Pad2): track 0.00 -> 39.0 mm
- net Net-(J9-Pad3): track 0.00 -> 35.4 mm
- net Net-(J9-Pad4): track 0.00 -> 31.8 mm
- net Net-(J10-Pad4): track 0.00 -> 25.6 mm
- net Net-(J10-Pad5): track 0.00 -> 24.1 mm
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- added copper zone on B.Cu, net GND
Other:
- board outline added: 66 x 134 mm
- net class Default: trace_width 0.25 -> 0.3
- board text added: "TO-220 screwed on the bottom of aluminum case (approximate position)."
